File: badge1.brd (EAGLE design)
At the start: 50 x 43.8 mm, 10 parts

Commit message: Rev 3 sent to Cogra
Parts:
- renumbered 1 to 6, 20150925 to 20151014
Other:
- board text added: "j.mp/iisbadge"
- board text removed: "tinyurl.com/iisbadge"
Changed lines of the file:
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@@
 <vertex x="6.25" y="37.5"/>
 </polygon>
-<text x="28.996834375" y="38.179075" size="1.016" layer="21" font="fixed">tinyurl.com/iisbadge</text>
+<text x="30.55589375" y="38.0923625" size="1.27" layer="21" font="fixed">j.mp/iisbadge</text>
 </plain>
 <attributes>
@@
 <element name="5" library="Discrete-new" package="LED2-2.54-D5.0MM" value="" x="42.75478125" y="27.944596875" rot="R90"/>
 <element name="RD@IIS.SE" library="SparkFun-Passives" package="AXIAL-0.4" value="" x="12.7" y="29.895" rot="R270"/>
-<element name="20150925" library="SparkFun-Passives" package="AXIAL-0.4" value="" x="15.24" y="29.895" rot="R270"/>
-<element name="1" library="wirepad" package="3,81/1,4" value="" x="25.025559375" y="33.660846875"/>
+<element name="20151014" library="SparkFun-Passives" package="AXIAL-0.4" value="" x="15.24" y="29.895" rot="R270"/>
+<element name="6" library="wirepad" package="3,81/1,4" value="" x="25.025559375" y="33.660846875"/>
 <element name="3" library="Seeed-OPL-Switch" package="SW6-2.54-9.0X3.5X3.2MM-90D" value="" x="25.029028125" y="6.343271875"/>
 <element name="GEEKPRT" library="SparkFun-Connectors" package="1X03_LOCK" value="" x="10.16" y="40.4301"/>
@@
 <signal name="N$5">
 <contactref element="3" pad="CH1B"/>
-<contactref element="20150925" pad="P$2"/>
+<contactref element="20151014" pad="P$2"/>
 <wire x1="26.289" y1="4.699" x2="27.559" y2="4.699" width="0.127" layer="16"/>
 <wire x1="23.876" y1="7.112" x2="26.289" y2="4.699" width="0.127" layer="16"/>
@@
 </signal>
 <signal name="N$7">
-<contactref element="20150925" pad="P$1"/>
+<contactref element="20151014" pad="P$1"/>
 <contactref element="GEEKPRT" pad="3"/>
 <wire x1="15.24" y1="40.5571" x2="15.24" y2="34.975" width="0.127" layer="1"/>
