File: rev3/badge1.brd (EAGLE design)
At the start: 50 x 43.8 mm, 10 parts

Commit message: Rev 3 sent to Cogra
Parts:
- removed U$2: (no value), logo:RECYCLING_10.00
- added U$1: (no value), OSHW:OSHW_6X200_NOTEXT
- moved U$3 23.9 mm to (28.3, 25.8)
- renumbered 1 to 6, 20150925 to 20151014
Routing:
- net GND: track 0.00 -> 56.2 mm
- net N$2: track 0.00 -> 29.7 mm
- net N$3: track 0.00 -> 29.1 mm
- net N$5: track 0.00 -> 27.0 mm
- net N$1: track 0.00 -> 25.8 mm
- net N$6: track 0.00 -> 23.4 mm
- net N$7: track 0.00 -> 5.58 mm
- net N$4: track 0.00 -> 5.33 mm
- added copper zone on layer 1, net GND
- added copper zone on layer 16, net GND
Other:
- board text added: "j.mp/iisbadge"
- board text removed: "http://tinyurl.com/iisbadge"
Changed lines of the file:
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@@
 <vertex x="6.25" y="37.5"/>
 </polygon>
-<text x="37.5" y="3.125" size="1.016" layer="1" font="vector">http://tinyurl.com/iisbadge</text>
+<text x="30.55589375" y="38.0923625" size="1.27" layer="21" font="fixed">j.mp/iisbadge</text>
 </plain>
 <attributes>
@@
 <element name="5" library="Discrete-new" package="LED2-2.54-D5.0MM" value="" x="42.75478125" y="27.944596875" rot="R90"/>
 <element name="RD@IIS.SE" library="SparkFun-Passives" package="AXIAL-0.4" value="" x="12.7" y="29.895" rot="R270"/>
-<element name="20150925" library="SparkFun-Passives" package="AXIAL-0.4" value="" x="15.24" y="29.895" rot="R270"/>
-<element name="1" library="wirepad" package="3,81/1,4" value="" x="25.025559375" y="33.660846875"/>
+<element name="20151014" library="SparkFun-Passives" package="AXIAL-0.4" value="" x="15.24" y="29.895" rot="R270"/>
+<element name="6" library="wirepad" package="3,81/1,4" value="" x="25.025559375" y="33.660846875"/>
 <element name="3" library="Seeed-OPL-Switch" package="SW6-2.54-9.0X3.5X3.2MM-90D" value="" x="25.029028125" y="6.343271875"/>
 <element name="GEEKPRT" library="SparkFun-Connectors" package="1X03_LOCK" value="" x="10.16" y="40.4301"/>
-<element name="U$2" library="logo" package="RECYCLING_10.00" value="" x="53.125" y="28.125"/>
-<element name="U$3" library="logo" package="MUELLTONNE_10.00" value="" x="50" y="15.625"/>
+<element name="U$3" library="logo" package="MUELLTONNE_10.00" value="" x="28.311315625" y="25.7688"/>
+<element name="U$1" library="OSHW" package="OSHW_6X200_NOTEXT" value="" x="39.996578125" y="31.45684375"/>
 </elements>
 <signals>
@@
 <contactref element="2" pad="-"/>
 <contactref element="GEEKPRT" pad="1"/>
-<wire x1="25.097659375" y1="18.601359375" x2="42.75478125" y2="29.214396875" width="0" layer="19" extent="1-1"/>
-<wire x1="7.72024375" y1="29.172446875" x2="25.097659375" y2="18.601359375" width="0" layer="19" extent="1-1"/>
-<wire x1="10.16" y1="40.5571" x2="7.72024375" y2="29.172446875" width="0" layer="19" extent="1-1"/>
+<wire x1="7.747" y1="38.1" x2="7.747" y2="29.21" width="0.127" layer="1"/>
+<wire x1="10.16" y1="40.513" x2="7.747" y2="38.1" width="0.127" layer="1"/>
+<wire x1="7.747" y1="29.21" x2="7.72024375" y2="29.172446875" width="0.127" layer="1"/>
+<wire x1="10.16" y1="40.513" x2="10.16" y2="40.5571" width="0.127" layer="1"/>
+<wire x1="35.687" y1="29.21" x2="42.672" y2="29.21" width="0.127" layer="1"/>
+<wire x1="25.146" y1="18.669" x2="35.687" y2="29.21" width="0.127" layer="1"/>
+<wire x1="42.672" y1="29.21" x2="42.75478125" y2="29.214396875" width="0.127" layer="1"/>
+<wire x1="25.146" y1="18.669" x2="25.097659375" y2="18.601359375" width="0.127" layer="1"/>
+<wire x1="14.605" y1="29.083" x2="7.747" y2="29.083" width="0.127" layer="1"/>
+<wire x1="25.019" y1="18.669" x2="14.605" y2="29.083" width="0.127" layer="1"/>
+<wire x1="7.747" y1="29.083" x2="7.72024375" y2="29.172446875" width="0.127" layer="1"/>
+<wire x1="25.019" y1="18.669" x2="25.097659375" y2="18.601359375" width="0.127" layer="1"/>
+<polygon width="0.4064" layer="1">
+<vertex x="-9.375" y="50"/>
+<vertex x="56.25" y="50"/>
+<vertex x="56.25" y="-3.125"/>
+<vertex x="-9.375" y="-3.125"/>
+</polygon>
+<polygon width="0.4064" layer="16">
+<vertex x="-12.5" y="53.125"/>
+<vertex x="56.25" y="53.125"/>
+<vertex x="56.25" y="50"/>
+<vertex x="56.25" y="-6.25"/>
+<vertex x="-12.5" y="-6.25"/>
+</polygon>
 </signal>
 <signal name="N$1">
 <contactref element="3" pad="COM2"/>
 <contactref element="4" pad="+"/>
-<wire x1="25.029028125" y1="7.993271875" x2="7.72024375" y2="26.632846875" width="0" layer="19" extent="1-1"/>
+<wire x1="25.019" y1="9.271" x2="25.019" y2="8.001" width="0.127" layer="1"/>
+<wire x1="7.747" y1="26.543" x2="25.019" y2="9.271" width="0.127" layer="1"/>
+<wire x1="25.019" y1="8.001" x2="25.029028125" y2="7.993271875" width="0.127" layer="1"/>
+<wire x1="7.747" y1="26.543" x2="7.72024375" y2="26.632846875" width="0.127" layer="1"/>
 </signal>
 <signal name="N$2">
 <contactref element="3" pad="COM1"/>
 <contactref element="5" pad="+"/>
-<wire x1="25.029028125" y1="4.693271875" x2="42.75478125" y2="26.674796875" width="0" layer="19" extent="1-1"/>
+<wire x1="25.527" y1="4.699" x2="25.146" y2="4.699" width="0.127" layer="1"/>
+<wire x1="42.672" y1="21.844" x2="25.527" y2="4.699" width="0.127" layer="1"/>
+<wire x1="42.672" y1="26.67" x2="42.672" y2="21.844" width="0.127" layer="1"/>
+<wire x1="25.146" y1="4.699" x2="25.029028125" y2="4.693271875" width="0.127" layer="1"/>
+<wire x1="42.672" y1="26.67" x2="42.75478125" y2="26.674796875" width="0.127" layer="1"/>
 </signal>
 <signal name="N$3">
@@
 <contactref element="2" pad="+1"/>
 <contactref element="3" pad="CH2A"/>
-<wire x1="18.366659375" y1="18.601359375" x2="31.828659375" y2="18.601359375" width="0" layer="19" extent="1-1"/>
-<wire x1="22.489028125" y1="7.993271875" x2="18.366659375" y2="18.601359375" width="0" layer="19" extent="1-1"/>
-<wire x1="22.489028125" y1="4.693271875" x2="22.489028125" y2="7.993271875" width="0" layer="19" extent="1-1"/>
+<wire x1="22.479" y1="7.874" x2="22.479" y2="4.699" width="0.127" layer="1"/>
+<wire x1="22.479" y1="4.699" x2="22.489028125" y2="4.693271875" width="0.127" layer="1"/>
+<wire x1="22.479" y1="7.874" x2="22.489028125" y2="7.993271875" width="0.127" layer="1"/>
+<wire x1="18.415" y1="12.065" x2="18.415" y2="18.542" width="0.127" layer="16"/>
+<wire x1="22.479" y1="8.001" x2="18.415" y2="12.065" width="0.127" layer="16"/>
+<wire x1="18.415" y1="18.542" x2="18.366659375" y2="18.601359375" width="0.127" layer="16"/>
+<wire x1="22.479" y1="8.001" x2="22.489028125" y2="7.993271875" width="0.127" layer="16"/>
+<wire x1="18.415" y1="18.669" x2="31.75" y2="18.669" width="0.127" layer="16"/>
+<wire x1="31.75" y1="18.669" x2="31.828659375" y2="18.601359375" width="0.127" layer="16"/>
+<wire x1="18.415" y1="18.669" x2="18.366659375" y2="18.601359375" width="0.127" layer="16"/>
 </signal>
 <signal name="N$5">
 <contactref element="3" pad="CH1B"/>
-<contactref element="20150925" pad="P$2"/>
-<wire x1="27.569028125" y1="4.693271875" x2="15.24" y2="24.815" width="0" layer="19" extent="1-1"/>
+<contactref element="20151014" pad="P$2"/>
+<wire x1="26.289" y1="4.699" x2="27.559" y2="4.699" width="0.127" layer="16"/>
+<wire x1="23.876" y1="7.112" x2="26.289" y2="4.699" width="0.127" layer="16"/>
+<wire x1="22.098" y1="7.112" x2="23.876" y2="7.112" width="0.127" layer="16"/>
+<wire x1="15.24" y1="13.97" x2="22.098" y2="7.112" width="0.127" layer="16"/>
+<wire x1="15.24" y1="24.815" x2="15.24" y2="13.97" width="0.127" layer="16"/>
+<wire x1="27.559" y1="4.699" x2="27.569028125" y2="4.693271875" width="0.127" layer="16"/>
 </signal>
 <signal name="N$6">
 <contactref element="3" pad="CH2B"/>
 <contactref element="RD@IIS.SE" pad="P$2"/>
-<wire x1="27.569028125" y1="7.993271875" x2="12.7" y2="24.815" width="0" layer="19" extent="1-1"/>
+<wire x1="26.797" y1="8.001" x2="27.559" y2="8.001" width="0.127" layer="1"/>
+<wire x1="12.7" y1="22.098" x2="26.797" y2="8.001" width="0.127" layer="1"/>
+<wire x1="12.7" y1="24.815" x2="12.7" y2="22.098" width="0.127" layer="1"/>
+<wire x1="27.559" y1="8.001" x2="27.569028125" y2="7.993271875" width="0.127" layer="1"/>
 </signal>
 <signal name="N$4">
 <contactref element="RD@IIS.SE" pad="P$1"/>
 <contactref element="GEEKPRT" pad="2"/>
-<wire x1="12.7" y1="40.3031" x2="12.7" y2="34.975" width="0" layer="19" extent="1-1"/>
+<wire x1="12.7" y1="40.3031" x2="12.7" y2="34.975" width="0.127" layer="1"/>
 </signal>
 <signal name="N$7">
-<contactref element="20150925" pad="P$1"/>
+<contactref element="20151014" pad="P$1"/>
 <contactref element="GEEKPRT" pad="3"/>
-<wire x1="15.24" y1="40.5571" x2="15.24" y2="34.975" width="0" layer="19" extent="1-1"/>
+<wire x1="15.24" y1="40.5571" x2="15.24" y2="34.975" width="0.127" layer="1"/>
 </signal>
 </signals>
